File: lasprema.sch (KiCad schematic (older format))
At the start: 108 parts, among them SW1 SW_PUSH, SW10 SW_PUSH, SW11 SW_PUSH, SW12 SW_PUSH, SW13 SW_PUSH, SW14 SW_PUSH, SW15 SW_PUSH, SW16 SW_PUSH, SW17 SW_PUSH, SW18 SW_PUSH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

Commit message: add case & confirm work perfect
Parts:
- U1: symbol promicro:ProMicro -> lasprema-rescue:ProMicro-promicro
Changed lines of the file:
@@
 $EndDescr
 $Comp
-L promicro:ProMicro U1
+L lasprema-rescue:ProMicro-promicro U1
 U 1 1 5CE4157F
 P 1600 1600
